Commit message: Update my_robot.xacro

File: catkin_ws/src/my_robot/urdf/my_robot.xacro (robot description, xacro)
@@ -63,5 +63,5 @@
       <origin xyz="-0.15 0 -0.05" rpy=" 0 0 0"/>
       <geometry>
-        <sphere radius="0.06"/>
+        <sphere radius="0.0599"/>
       </geometry>
     </collision>
@@ -69,5 +69,5 @@
       <origin xyz="-0.15 0 -0.05" rpy=" 0 0 0"/>
       <geometry>
-        <sphere radius="0.06"/>
+        <sphere radius="0.0599"/>
       </geometry>
     </visual>
@@ -75,5 +75,5 @@
       <origin xyz="0.15 0 -0.05" rpy=" 0 0 0"/>
       <geometry>
-        <sphere radius="0.06"/>
+        <sphere radius="0.0599"/>
       </geometry>
     </collision>
@@ -81,5 +81,5 @@
       <origin xyz="0.15 0 -0.05" rpy=" 0 0 0"/>
       <geometry>
-        <sphere radius="0.06"/>
+        <sphere radius="0.0599"/>
       </geometry>
     </visual>
@@ -94,5 +94,5 @@
       <origin xyz="0.0 0.0 0.0" rpy="0.0 1.5707 1.5707"/>
       <geometry>
-        <cylinder radius="0.115" length="0.06"/>
+        <cylinder radius="0.11" length="0.06"/>
       </geometry>
       <material name="">
@@ -104,5 +104,5 @@
       <origin xyz="0.0 0.0 0.0" rpy="0.0 1.5707 1.5707"/>
       <geometry>
-        <cylinder radius="0.115" length="0.06"/>
+        <cylinder radius="0.11" length="0.06"/>
       </geometry>
     </collision>
@@ -117,5 +117,5 @@
       <origin xyz="0.0 0.0 0.0" rpy="0.0 1.5707 1.5707"/>
       <geometry>
-        <cylinder radius="0.115" length="0.06"/>
+        <cylinder radius="0.11" length="0.06"/>
       </geometry>
       <material name="">
@@ -127,5 +127,5 @@
       <origin xyz="0.0 0.0 0.0" rpy="0.0 1.5707 1.5707"/>
       <geometry>
-        <cylinder radius="0.115" length="0.06"/>
+        <cylinder radius="0.11" length="0.06"/>
       </geometry>
     </collision>
